File: Hardware/Electronics/CAD/CatDoor.sch (KiCad schematic (older format))
At the start: 5 parts, among them J1 MPE 094-1-006, SW1 SS ESP101, SW2 SW_DPST_x2, U4 ESP-12E

Commit message: library linkage fix
Parts:
- removed SW1: SS ESP101, Switch:ESP20XX, symbol SW_DPDT_x2
- added J?: MPE 094-1-003, symbol CONN_01X03
- SW2: value SW_DPST_x2 -> SMD 4x4mm Button
Connections:
- wire segments 27 -> 31
Other:
- moved on the sheet: SW2A
Changed lines of the file:
@@
 LIBS:valves
 LIBS:ESP8266
-LIBS:HILINK
-LIBS:SSR
-LIBS:switches
+LIBS:HiLink
 LIBS:L9110
-LIBS:pololu_a4988
-LIBS:iot_cat_door-cache
+LIBS:SW_DPST_x2
 EELAYER 25 0
 EELAYER END
@@
 NoConn ~ 3000 1275
 NoConn ~ 3000 1675
-$Comp
-L SW_DPDT_x2 SW1
-U 1 1 592C5A5F
-P 2875 2525
-F 0 "SW1" H 2750 2800 50  0000 C CNN
-F 1 "SS ESP101" H 2875 2725 50  0000 C CNN
-F 2 "Switch:ESP20XX" H 2875 2525 50  0001 C CNN
-F 3 "" H 2875 2525 50  0001 C CNN
-	1    2875 2525
-	1    0    0    -1
-$EndComp
-Text GLabel 2525 2525 0    60   Input ~ 0
+Text GLabel 3000 2400 2    60   Input ~ 0
 MODE
 $Comp
 L GND #PWR09
 U 1 1 592C5F8F
-P 3175 2425
-F 0 "#PWR09" H 3175 2175 50  0001 C CNN
-F 1 "GND" V 3225 2275 50  0000 C CNN
-F 2 "" H 3175 2425 50  0001 C CNN
-F 3 "" H 3175 2425 50  0001 C CNN
-	1    3175 2425
+P 3025 2200
+F 0 "#PWR09" H 3025 1950 50  0001 C CNN
+F 1 "GND" V 3075 2050 50  0000 C CNN
+F 2 "" H 3025 2200 50  0001 C CNN
+F 3 "" H 3025 2200 50  0001 C CNN
+	1    3025 2200
 	0    -1   -1   0
 $EndComp
@@
 L +3.3V #PWR010
 U 1 1 592C600F
-P 3175 2625
-F 0 "#PWR010" H 3175 2475 50  0001 C CNN
-F 1 "+3.3V" V 3225 2800 50  0000 C CNN
-F 2 "" H 3175 2625 50  0001 C CNN
-F 3 "" H 3175 2625 50  0001 C CNN
-	1    3175 2625
+P 3025 2600
+F 0 "#PWR010" H 3025 2450 50  0001 C CNN
+F 1 "+3.3V" V 3075 2775 50  0000 C CNN
+F 2 "" H 3025 2600 50  0001 C CNN
+F 3 "" H 3025 2600 50  0001 C CNN
+	1    3025 2600
 	0    1    1    0
 $EndComp
@@
 L SW_DPST_x2 SW2
 U 1 1 599EBC5A
-P 2450 3200
-F 0 "SW2" H 2450 3100 50  0000 C CNN
-F 1 "SW_DPST_x2" H 2450 3000 50  0000 C CNN
-F 2 "Buttons_Switches_SMD:SW_SPST_SKQG" H 2450 3200 50  0001 C CNN
-F 3 "" H 2450 3200 50  0001 C CNN
-	1    2450 3200
+P 2300 3200
+F 0 "SW2" H 2300 3100 50  0000 C CNN
+F 1 "SMD 4x4mm Button" H 2300 3000 50  0000 C CNN
+F 2 "Buttons_Switches_SMD:SW_SPST_SKQG" H 2300 3200 50  0001 C CNN
+F 3 "" H 2300 3200 50  0001 C CNN
+	1    2300 3200
 	1    0    0    -1
 $EndComp
@@
 L +3.3V #PWR012
 U 1 1 599EBD49
-P 2100 3200
-F 0 "#PWR012" H 2100 3050 50  0001 C CNN
-F 1 "+3.3V" V 2100 3450 50  0000 C CNN
-F 2 "" H 2100 3200 50  0001 C CNN
-F 3 "" H 2100 3200 50  0001 C CNN
-	1    2100 3200
+P 1800 3200
+F 0 "#PWR012" H 1800 3050 50  0001 C CNN
+F 1 "+3.3V" V 1800 3450 50  0000 C CNN
+F 2 "" H 1800 3200 50  0001 C CNN
+F 3 "" H 1800 3200 50  0001 C CNN
+	1    1800 3200
 	0    -1   -1   0
 $EndComp
@@
 	3000 1775 2850 1775
 Wire Wire Line
-	3075 2425 3175 2425
-Wire Wire Line
-	3175 2625 3075 2625
-Wire Wire Line
-	2675 2525 2525 2525
+	2825 2200 3025 2200
+Wire Wire Line
+	2825 2600 3025 2600
+Wire Wire Line
+	2725 2400 3000 2400
 Wire Wire Line
 	8500 1975 9050 1975
 Wire Wire Line
-	2100 3200 2250 3200
+	1800 3200 1950 3200
 Wire Wire Line
 	3150 3350 3300 3350
@@
 Wire Wire Line
 	9050 1775 8500 1775
+$Comp
+L CONN_01X03 J?
+U 1 1 5B8D803F
+P 2525 2400
+F 0 "J?" H 2525 2600 50  0000 C CNN
+F 1 "MPE 094-1-003" V 2625 2400 50  0000 C CNN
+F 2 "" H 2525 2400 50  0001 C CNN
+F 3 "" H 2525 2400 50  0001 C CNN
+	1    2525 2400
+	-1   0    0    1
+$EndComp
+Wire Wire Line
+	2825 2600 2825 2500
+Wire Wire Line
+	2825 2500 2725 2500
+Wire Wire Line
+	2725 2300 2825 2300
+Wire Wire Line
+	2825 2300 2825 2200
 $EndSCHEMATC
